Commit message: update lite urdf

File: lite_urdf_publish/urdf/humanoid_publish.urdf (robot description, URDF)
Before this commit: robot humanoid, 22 links, 21 joints
Joints:
- joint hip_roll_l_joint: origin xyz=0 0.13 -0.0659230484541305 rpy=0 0 0 -> xyz=0 0.13 -0.079 rpy=0 0 0
- joint hip_roll_r_joint: origin xyz=0 -0.13 -0.0659230484541306 rpy=0 0 0 -> xyz=0 -0.13 -0.079 rpy=0 0 0

Commit message: update lite urdf

File: lite_urdf_publish/urdf/humanoid_publish.urdf (robot description, URDF)
Before this commit: robot humanoid, 22 links, 21 joints
Joints:
- joint waist_joint: origin xyz=0 0 0.0192 rpy=0 0 0 -> xyz=0 0 0.006 rpy=0 0 0
